File: MIPI Board 5/MIPIBoard5/MIPIBoard5.kicad_pcb (KiCad board)
At the start: 4 copper layers, 55.2 x 46.7 mm, 69 parts, among them J1 Power/Control Top, J2 Bank A Top, J3 Bank B Top, J4 MIPI1, J5 MIPI2, J6 Bank A Bottom, J7 Bank B Bottom, J8 Power/Control Bottom, U1 LM339, U2 LM339, U3 LM339, U4 TLV3605RVKR, U5 TLV3605RVKR, U6 TLV3605RVKR, U7 TLV3605RVKR, U8 TLV3605RVKR, U9 TLV3605RVKR

Commit message: fixed small errors
Routing:
- net +3V3: track 238.7 -> 252.2 mm, vias 5 -> 4
- net 34_L3/1.5B_N: track 50.6 -> 51.3 mm
- net Cam1_D0_P: vias 3 -> 2
- net Cam1_D0_N: vias 4 -> 3
- net Cam1_CK_N: vias 1 -> 0
Changed lines of the file:
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@@
 	)
 	(segment
+		(start 93.799748 76.49)
+		(end 93.779748 76.47)
+		(width 0.4)
+		(layer "F.Cu")
+		(net "+3V3")
+	)
+	(segment
 		(start 71.05 61.2)
 		(end 72.05 60.2)
@@
 	)
 	(segment
+		(start 85.62 76.47)
+		(end 84.85 75.7)
+		(width 0.4)
+		(layer "F.Cu")
+		(net "+3V3")
+	)
+	(segment
 		(start 93.799748 81.1632)
 		(end 93.799748 82.350252)
@@
 	)
 	(segment
+		(start 72.830076 70.8)
+		(end 70.6 70.8)
+		(width 0.4)
+		(layer "F.Cu")
+		(net "+3V3")
+	)
+	(segment
 		(start 60 84.025)
 		(end 59.9 83.925)
@@
 	)
 	(segment
+		(start 73.040076 70.59)
+		(end 72.830076 70.8)
+		(width 0.4)
+		(layer "F.Cu")
+		(net "+3V3")
+	)
+	(segment
 		(start 72.05 60.2)
 		(end 76.3 60.2)
@@
 	)
 	(segment
+		(start 93.779748 76.47)
+		(end 85.62 76.47)
+		(width 0.4)
+		(layer "F.Cu")
+		(net "+3V3")
+	)
+	(segment
 		(start 70.6 70.15)
-		(end 70.6 71.457228)
+		(end 70.6 70.8)
 		(width 0.6)
 		(layer "F.Cu")
@@
 	)
 	(segment
+		(start 70.6 70.8)
+		(end 70.6 71.457228)
+		(width 0.6)
+		(layer "F.Cu")
+		(net "+3V3")
+	)
+	(segment
 		(start 94.8 68.816674)
 		(end 94.8 67.3)
@@
 	)
 	(segment
+		(start 74.8 70.59)
+		(end 73.040076 70.59)
+		(width 0.4)
+		(layer "F.Cu")
+		(net "+3V3")
+	)
+	(segment
 		(start 85.8 63.45)
 		(end 85.8 67.65)
@@
 	)
 	(via
-		(at 56.91 79.5)
-		(size 0.6)
-		(drill 0.3)
-		(layers "F.Cu" "B.Cu")
-		(net "+3V3")
-	)
-	(via
 		(at 93.45 82.7)
 		(size 0.6)
@@
 	)
 	(segment
-		(start 66.66 88.457366)
+		(start 67.200943 86.890249)
+		(end 66.9 86.890249)
+		(width 0.16)
+		(layer "B.Cu")
+		(net "34_L3{slash}1.5B_N")
+	)
+	(segment
+		(start 67.440949 85.330249)
+		(end 67.440949 85.450249)
+		(width 0.16)
+		(layer "B.Cu")
+		(net "34_L3{slash}1.5B_N")
+	)
+	(segment
+		(start 67.200949 85.690249)
+		(end 66.9 85.690249)
+		(width 0.16)
+		(layer "B.Cu")
+		(net "34_L3{slash}1.5B_N")
+	)
+	(segment
+		(start 66.66 89.288882)
 		(end 66.66 92.633725)
 		(width 0.16)
@@
 	)
 	(segment
-		(start 66.66 76.833726)
-		(end 66.66 86.063)
+		(start 66.66 85.930249)
+		(end 66.66 86.050249)
 		(width 0.16)
 		(layer "B.Cu")
@@
 	)
 	(segment
-		(start 66.66 92.633725)
-		(end 67.757574 93.731299)
+		(start 66.66 76.833726)
+		(end 66.66 84.850249)
 		(width 0.16)
 		(layer "B.Cu")
@@
 	)
 	(segment
-		(start 67.757574 93.731299)
-		(end 68.068701 93.731299)
+		(start 66.9 85.090249)
+		(end 67.200949 85.090249)
+		(width 0.16)
+		(layer "B.Cu")
+		(net "34_L3{slash}1.5B_N")
+	)
+	(segment
+		(start 67.440943 86.530249)
+		(end 67.440943 86.650249)
+		(width 0.16)
+		(layer "B.Cu")
+		(net "34_L3{slash}1.5B_N")
+	)
+	(segment
+		(start 65.426274 75.6)
+		(end 66.66 76.833726)
 		(width 0.16)
 		(layer "B.Cu")
@@
 	)
 	(segment
-		(start 67.42 86.903)
-		(end 66.9 86.903)
+		(start 65.2 75.6)
+		(end 65.426274 75.6)
 		(width 0.16)
 		(layer "B.Cu")
@@
 	)
 	(segment
-		(start 65.426274 75.6)
-		(end 66.66 76.833726)
+		(start 66.66 87.130249)
+		(end 66.66 87.250249)
 		(width 0.16)
 		(layer "B.Cu")
@@
 	)
 	(segment
-		(start 65.2 75.6)
-		(end 65.426274 75.6)
+		(start 66.66 92.633725)
+		(end 67.757574 93.731299)
 		(width 0.16)
 		(layer "B.Cu")
@@
 	)
 	(segment
-		(start 66.66 87.143)
-		(end 66.66 87.263)
+		(start 66.9 86.290249)
+		(end 67.200943 86.290249)
 		(width 0.16)
 		(layer "B.Cu")
@@
 	)
 	(segment
-		(start 66.9 86.303)
-		(end 67.42 86.303)
+		(start 66.66 87.250249)
+		(end 66.66 89.288882)
 		(width 0.16)
 		(layer "B.Cu")
@@
 	)
 	(segment
-		(start 67.66 86.543)
-		(end 67.66 86.663)
+		(start 67.757574 93.731299)
+		(end 68.068701 93.731299)
 		(width 0.16)
 		(layer "B.Cu")
 		(net "34_L3{slash}1.5B_N")
 	)
-	(segment
-		(start 66.66 87.263)
-		(end 66.66 88.457366)
+	(arc
+		(start 67.200949 85.090249)
+		(mid 67.370655 85.160543)
+		(end 67.440949 85.330249)
+		(width 0.16)
+		(layer "B.Cu")
+		(net "34_L3{slash}1.5B_N")
+	)
+	(arc
+		(start 67.440943 86.650249)
+		(mid 67.370649 86.819955)
+		(end 67.200943 86.890249)
 		(width 0.16)
 		(layer "B.Cu")
@@
 	)
 	(arc
-		(start 66.9 86.903)
-		(mid 66.730294 86.973294)
-		(end 66.66 87.143)
+		(start 66.9 86.890249)
+		(mid 66.730294 86.960543)
+		(end 66.66 87.130249)
 		(width 0.16)
 		(layer "B.Cu")
@@
 	)
 	(arc
-		(start 67.66 86.663)
-		(mid 67.589706 86.832706)
-		(end 67.42 86.903)
+		(start 67.200943 86.290249)
+		(mid 67.370649 86.360543)
+		(end 67.440943 86.530249)
 		(width 0.16)
 		(layer "B.Cu")
@@
 	)
 	(arc
-		(start 66.66 86.063)
-		(mid 66.730294 86.232706)
-		(end 66.9 86.303)
+		(start 66.9 85.690249)
+		(mid 66.730294 85.760543)
+		(end 66.66 85.930249)
 		(width 0.16)
 		(layer "B.Cu")
@@
 	)
 	(arc
-		(start 67.42 86.303)
-		(mid 67.589706 86.373294)
-		(end 67.66 86.543)
+		(start 67.440949 85.450249)
+		(mid 67.370655 85.619955)
+		(end 67.200949 85.690249)
+		(width 0.16)
+		(layer "B.Cu")
+		(net "34_L3{slash}1.5B_N")
+	)
+	(arc
+		(start 66.66 86.050249)
+		(mid 66.730294 86.219955)
+		(end 66.9 86.290249)
+		(width 0.16)
+		(layer "B.Cu")
+		(net "34_L3{slash}1.5B_N")
+	)
+	(arc
+		(start 66.66 84.850249)
+		(mid 66.730294 85.019955)
+		(end 66.9 85.090249)
 		(width 0.16)
 		(layer "B.Cu")
@@
 		(net "Cam1_CK_N")
 	)
-	(via
-		(at 56.91 72.5)
-		(size 0.6)
-		(drill 0.3)
-		(layers "F.Cu" "B.Cu")
-		(net "Cam1_CK_N")
-	)
 	(segment
 		(start 74.787669 65.8)
@@
 	)
 	(via
-		(at 68.8 65.8)
-		(size 0.6)
-		(drill 0.3)
-		(layers "F.Cu" "B.Cu")
-		(net "Cam1_D0_P")
-	)
-	(via
 		(at 71.28 65.8)
 		(size 0.6)
@@
 	)
 	(via
-		(at 68.8 64.5)
-		(size 0.6)
-		(drill 0.3)
-		(layers "F.Cu" "B.Cu")
-		(net "Cam1_D0_N")
-	)
-	(via
 		(at 56.91 66.5)
 		(size 0.6)
@@
 		(base_line
 			(pts
-				(xy 66.66 86.063) (xy 66.66 88.457366)
+				(xy 66.66 84.850249) (xy 66.66 89.288882)
+			)
+		)
+		(base_line_coupled
+			(pts
+				(xy 66.34 84.850249) (xy 66.34 84.831677)
 			)
 		)
 		(corner_radius_percent 80)
 		(end
-			(xy 66.66 88.457366)
+			(xy 66.66 89.288882)
 		)
 		(initial_side "left")
@@
 		(last_status "tuned")
 		(last_track_width 0.16)
-		(last_tuning_length 55.373538)
+		(last_tuning_length -1.7e-05)
 		(max_amplitude 1)
 		(min_amplitude 0.2)
 		(min_spacing 0.6)
 		(origin
-			(xy 66.66 86.063)
+			(xy 66.66 84.850249)
 		)
 		(override_custom_rules no)
@@
 		(target_skew_max 0.1)
 		(target_skew_min -0.1)
-		(tuning_mode "single")
-		(members "051baa5d-b9f3-4bea-9579-1cbaf8c9ba97" "9e792fbd-6c2c-4650-9f7d-42c2ca22c1b1"
-			"9f420136-977b-4089-8cc7-ffebfcbef191" "a7ec96fe-6e6e-4e24-8b59-832fb855c018"
-			"b34789e7-fb23-4f91-a974-004226a20346" "d7b196b6-93c0-4b3e-a203-d86ffa305e3d"
-			"dd248413-d073-4ee1-8c28-89255b48cd10" "e6c72a0c-7e6d-4bf2-adf8-cab8f6223859"
-			"f7909ed9-07bb-41fe-a7ad-b1fbb6cc1302"
+		(tuning_mode "diff_pair_skew")
+		(members "0335e565-f3c5-443b-9253-13cdd64498e0" "091602a3-7943-4cea-9536-ebbda2fe9d56"
+			"1ebfcb99-4e71-443d-9981-9f412475f9f5" "2281ffdb-b1d3-4b7f-8586-a67114250f67"
+			"333f9327-1bcf-46d1-82bf-924a31b76d95" "4252653f-016e-4710-bfe1-c568aa682aae"
+			"4de7b4df-c3f2-406c-b690-7f571c1c0b18" "65352a01-338f-45ad-af85-61ece2d45a03"
+			"69573755-63e7-4eb1-91f0-d0b4e69aa97e" "73eb0b74-23de-482c-ab7f-a098f73d3d01"
+			"a65fc927-7420-4877-bb33-93532a0c579b" "ab9dd5ca-a148-4933-a6bd-497caab3b469"
+			"c50e31fa-dfaa-48cd-b5a7-78d48331005f" "d6143492-5abc-4d53-8faa-bf278c541c1d"
+			"ddd26a5c-c324-44e1-a4fa-fbe46bd25715" "e0b77d1e-36bb-4c14-85ca-82d30fc01202"
+			"e60d8978-62f0-4c5f-abd6-ed275efafd17"
 		)
 	)
